Commit message: Using body v3 and joint Constraint

File: urdf/caster_moma_j2n6s200_xacro_standard.xacro (robot description, xacro)
@@ -7,5 +7,5 @@
   <xacro:include filename = "$(find caster_description)/urdf/body/caster_body_v3.urdf.xacro" />
   <!-- sensor include -->
-  <xacro:include filename="$(find caster_moma_description)/urdf/kinova/j2n6s200.xacro" />
+  <xacro:include filename="$(find kinova_description)/urdf/j2n6s200.xacro" />
   <xacro:include filename="$(find pan_tilt_description)/urdf/pan_tilt.urdf.xacro" />
   <xacro:include filename="$(find pan_tilt_description)/urdf/kinect_v2.urdf.xacro" />

File: urdf/caster_moma_j2s6s200_xacro.xacro (robot description, xacro)
@@ -5,7 +5,7 @@
   <xacro:include filename = "$(find caster_description)/urdf/common_properties.xacro" />
   <xacro:include filename = "$(find caster_description)/urdf/caster_v2.urdf.xacro" />
-  <xacro:include filename = "$(find caster_description)/urdf/body/caster_body_v2.urdf.xacro" />
+  <xacro:include filename = "$(find caster_description)/urdf/body/caster_body_v3.urdf.xacro" />
   <!-- sensor include -->
-  <xacro:include filename="$(find kinova_description)/urdf/j2s6s200.xacro" />
+  <xacro:include filename="$(find caster_moma_description)/urdf/kinova/j2s6s200.xacro" />
   <xacro:include filename="$(find pan_tilt_description)/urdf/pan_tilt.urdf.xacro" />
   <xacro:include filename="$(find pan_tilt_description)/urdf/kinect_v2.urdf.xacro" />
@@ -14,5 +14,5 @@
   <caster_robot/>
   <xacro:caster_body parent="base_link">
-    <origin xyz="0.072 0.0 0.2815" rpy="0 0 0" />
+    <origin xyz="0.0 0.0 0.266" rpy="0 0 0" />
   </xacro:caster_body>
    <!-- realsense d435 -->
@@ -21,6 +21,7 @@
   <link name="arm_mount_link" />
   <joint name="arm_mount_joint" type="fixed">
-    <origin xyz="0 0 0" rpy="${M_PI/2} 0 0" />
-    <parent link="caster_body_arm_link"/>
+    <origin xyz="0.076 0.0 -0.031" rpy="0 0 ${M_PI}" />
+    <!-- <origin xyz="0.072 0.001 0.1465" rpy="0 0 0" /> -->
+    <parent link="caster_body_arm_mount_link"/>
     <child link="arm_mount_link"/>
   </joint>
@@ -51,5 +52,5 @@
   </xacro:pan_tilt_neck_50mm> -->
   <xacro:pan_tilt parent="caster_body_head_link" >
-    <origin xyz="0 0 0" rpy="0 0 0" />
+    <origin xyz="-0.0266 0 0" rpy="0 0 0" />
   </xacro:pan_tilt>
   <!-- kinect -->

File: urdf/caster_moma_j2s6s200_xacro_standard.xacro (robot description, xacro)
@@ -7,5 +7,5 @@
   <xacro:include filename = "$(find caster_description)/urdf/body/caster_body_v3.urdf.xacro" />
   <!-- sensor include -->
-  <xacro:include filename="$(find caster_moma_description)/urdf/kinova/j2n6s200.xacro" />
+  <xacro:include filename="$(find kinova_description)/urdf/j2s6s200.xacro" />
   <xacro:include filename="$(find pan_tilt_description)/urdf/pan_tilt.urdf.xacro" />
   <xacro:include filename="$(find pan_tilt_description)/urdf/kinect_v2.urdf.xacro" />
@@ -26,5 +26,5 @@
     <child link="arm_mount_link"/>
   </joint>
-  <xacro:j2n6s200 base_parent="arm_mount_link"/>
+  <xacro:j2s6s200 base_parent="arm_mount_link"/>
   <!-- realsense -->
   <link name="realsense_coupling_link">
@@ -41,5 +41,5 @@
   <joint name="realsense_coupling_joint" type="fixed">
     <origin xyz="0 0 0.007" rpy="0 0 0" />
-    <parent link="j2n6s200_link_6"/>
+    <parent link="j2s6s200_link_6"/>
     <child link="realsense_coupling_link"/>
   </joint>
